File: _autosave-Flatbox-rev5.kicad_sch (KiCad schematic)
At the start: 24 parts, among them SW1 SW_Push, SW10 SW_Push, SW11 SW_Push, SW12 SW_Push, SW13 SW_Push, SW14 SW_Push, SW15 SW_Push, SW16 SW_Push, SW17 SW_Push, SW18 SW_Push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

Commit message: PUSH
Connections:
- net GND: now also SW10.2, SW7.2; no longer SW10.1, SW7.1
- net LEFT: now also SW7.1; no longer SW7.2
- net SQUARE: now also SW10.1; no longer SW10.2
Other:
- moved on the sheet: SW10, SW11, SW12, SW13, SW14, SW15, SW16, SW17, SW18, SW8, SW9
